File: board_hab2/HAB.brd (EAGLE design)
At the start: 120.3 x 101.6 mm, 31 parts

Commit message: updated gitignore and added comments to HAB board
Parts:
- removed THROUGH_HOLE_AMBIENT_TEMP_SENSOR: SSW-103-02-S-S, con-samtec:SSW-103-02-S-S
- added T2: 2N3904, transistor:TO92
Connections:
- new net N$27: JP11.2
- new net N$28: B1.A6, T2.2
- new net N$29: B1.3.3V
- net 5V: no longer JP11.2
- net GND: now also T2.1; no longer THROUGH_HOLE_AMBIENT_TEMP_SENSOR.3
- net N$24: no longer THROUGH_HOLE_AMBIENT_TEMP_SENSOR.2
- net N$25: now also T2.3; no longer THROUGH_HOLE_AMBIENT_TEMP_SENSOR.1
Changed lines of the file:
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@@
 <?xml version="1.0" encoding="utf-8"?>
 <!DOCTYPE eagle SYSTEM "eagle.dtd">
-<eagle version="8.3.2">
+<eagle version="8.7.1">
 <drawing>
 <settings>
@@
 <layers>
 <layer number="1" name="Top" color="4" fill="1" visible="yes" active="yes"/>
+<layer number="2" name="Route2" color="1" fill="3" visible="no" active="yes"/>
+<layer number="3" name="Route3" color="4" fill="3" visible="no" active="yes"/>
+<layer number="4" name="Route4" color="1" fill="4" visible="no" active="yes"/>
+<layer number="5" name="Route5" color="4" fill="4" visible="no" active="yes"/>
+<layer number="6" name="Route6" color="1" fill="8" visible="no" active="yes"/>
+<layer number="7" name="Route7" color="4" fill="8" visible="no" active="yes"/>
+<layer number="8" name="Route8" color="1" fill="2" visible="no" active="yes"/>
+<layer number="9" name="Route9" color="4" fill="2" visible="no" active="yes"/>
+<layer number="10" name="Route10" color="1" fill="7" visible="no" active="yes"/>
+<layer number="11" name="Route11" color="4" fill="7" visible="no" active="yes"/>
+<layer number="12" name="Route12" color="1" fill="5" visible="no" active="yes"/>
+<layer number="13" name="Route13" color="4" fill="5" visible="no" active="yes"/>
+<layer number="14" name="Route14" color="1" fill="6" visible="no" active="yes"/>
+<layer number="15" name="Route15" color="4" fill="6" visible="no" active="yes"/>
 <layer number="16" name="Bottom" color="1" fill="1" visible="yes" active="yes"/>
 <layer number="17" name="Pads" color="2" fill="1" visible="yes" active="yes"/>
@@
 <param name="dpMaxLengthDifference" value="10mm"/>
 <param name="dpGapFactor" value="2.5"/>
-<param name="checkGrid" value="0"/>
 <param name="checkAngle" value="0"/>
 <param name="checkFont" value="1"/>
 <param name="checkRestrict" value="1"/>
+<param name="checkStop" value="0"/>
+<param name="checkValues" value="0"/>
 <param name="useDiameter" value="13"/>
 <param name="maxErrors" value="50"/>
@@
 <attribute name="OC_NEWARK" value="unknown" x="86.36" y="78.74" size="1.778" layer="27" display="off"/>
 </element>
-<element name="THROUGH_HOLE_AMBIENT_TEMP_SENSOR" library="con-samtec" library_urn="urn:adsk.eagle:library:184" package="SSW-103-02-S-S" value="SSW-103-02-S-S" x="11.43" y="80.01">
-<attribute name="MF" value="" x="11.43" y="80.01" size="1.778" layer="27" display="off"/>
-<attribute name="MPN" value="SSW-103-02-S-S" x="11.43" y="80.01" size="1.778" layer="27" display="off"/>
-<attribute name="OC_FARNELL" value="unknown" x="11.43" y="80.01" size="1.778" layer="27" display="off"/>
-<attribute name="OC_NEWARK" value="11P9367" x="11.43" y="80.01" size="1.778" layer="27" display="off"/>
-</element>
 <element name="JP11" library="jumper" library_urn="urn:adsk.eagle:library:252" package="JP1" package3d_urn="urn:adsk.eagle:package:15455/1" value="" x="80.01" y="3.81"/>
+<element name="T2" library="transistor" library_urn="urn:adsk.eagle:library:402" package="TO92" package3d_urn="urn:adsk.eagle:package:29893/2" value="2N3904" x="-8.89" y="-33.02"/>
 </elements>
 <signals>
@@
 <wire x1="59.7951125" y1="49.53" x2="55.7567125" y2="45.4916" width="0.3048" layer="16"/>
 <contactref element="I2C_CLK" pad="1"/>
-<wire x1="33.02" y1="22.86" x2="30.48" y2="25.4" width="0" layer="19" extent="1-16"/>
 <wire x1="33.02" y1="22.86" x2="36.83" y2="19.05" width="0.254" layer="16"/>
 <wire x1="36.83" y1="19.05" x2="36.83" y2="10.16" width="0.254" layer="16"/>
@@
 <contactref element="AMBIENT_TEMP_SENSOR" pad="3"/>
 <contactref element="TRACKSOAR" pad="1"/>
-<contactref element="THROUGH_HOLE_AMBIENT_TEMP_SENSOR" pad="3"/>
 <wire x1="58.42" y1="73.66" x2="57.15" y2="74.93" width="0.254" layer="16"/>
 <wire x1="57.15" y1="74.93" x2="56.59948125" y2="74.93" width="0.254" layer="16"/>
@@
 <wire x1="24.13" y1="40.64" x2="13.97" y2="40.64" width="0.254" layer="16"/>
 <wire x1="13.97" y1="40.64" x2="11.43" y2="38.1" width="0.254" layer="16"/>
+<contactref element="T2" pad="1"/>
 <wire x1="81.28" y1="78.74" x2="86.36" y2="85.09" width="0" layer="19" extent="1-1"/>
 <wire x1="58.42" y1="73.66" x2="81.28" y2="78.74" width="0" layer="19" extent="1-1"/>
@@
 <wire x1="48.26" y1="86.36" x2="43.18" y2="81.28" width="0" layer="19" extent="1-1"/>
 <wire x1="26.67" y1="85.09" x2="35.8902" y2="75.2602" width="0" layer="19" extent="16-16"/>
-<wire x1="13.97" y1="80.01" x2="26.67" y2="85.09" width="0" layer="19" extent="1-1"/>
 <wire x1="24.13" y1="40.64" x2="34.29" y2="73.66" width="0" layer="19" extent="16-16"/>
 <wire x1="66.04" y1="38.1" x2="58.42" y2="73.66" width="0" layer="19" extent="1-1"/>
+<wire x1="-7.62" y1="-33.02" x2="5.08" y2="10.16" width="0" layer="19" extent="1-1"/>
 </signal>
 <signal name="5V">
@@
 <contactref element="JP9" pad="1"/>
 <contactref element="JP10" pad="1"/>
-<contactref element="JP11" pad="2"/>
-<wire x1="17.78" y1="5.08" x2="80.01" y2="5.08" width="0" layer="19" extent="1-1"/>
-<wire x1="24.13" y1="5.08" x2="17.78" y2="5.08" width="0" layer="19" extent="1-1"/>
-<wire x1="30.48" y1="5.08" x2="24.13" y2="5.08" width="0" layer="19" extent="1-1"/>
-<wire x1="36.83" y1="5.08" x2="30.48" y2="5.08" width="0" layer="19" extent="1-1"/>
-<wire x1="43.18" y1="5.08" x2="36.83" y2="5.08" width="0" layer="19" extent="1-1"/>
-<wire x1="49.53" y1="5.08" x2="43.18" y2="5.08" width="0" layer="19" extent="1-1"/>
-<wire x1="55.88" y1="5.08" x2="49.53" y2="5.08" width="0" layer="19" extent="1-1"/>
-<wire x1="62.23" y1="2.54" x2="55.88" y2="5.08" width="0" layer="19" extent="1-1"/>
-<wire x1="68.58" y1="2.54" x2="62.23" y2="2.54" width="0" layer="19" extent="1-1"/>
-<wire x1="74.93" y1="2.54" x2="68.58" y2="2.54" width="0" layer="19" extent="1-1"/>
+<wire x1="68.58" y1="2.54" x2="74.93" y2="2.54" width="0" layer="19" extent="1-1"/>
+<wire x1="62.23" y1="2.54" x2="68.58" y2="2.54" width="0" layer="19" extent="1-1"/>
+<wire x1="55.88" y1="5.08" x2="62.23" y2="2.54" width="0" layer="19" extent="1-1"/>
+<wire x1="49.53" y1="5.08" x2="55.88" y2="5.08" width="0" layer="19" extent="1-1"/>
+<wire x1="43.18" y1="5.08" x2="49.53" y2="5.08" width="0" layer="19" extent="1-1"/>
+<wire x1="36.83" y1="5.08" x2="43.18" y2="5.08" width="0" layer="19" extent="1-1"/>
+<wire x1="30.48" y1="5.08" x2="36.83" y2="5.08" width="0" layer="19" extent="1-1"/>
+<wire x1="24.13" y1="5.08" x2="30.48" y2="5.08" width="0" layer="19" extent="1-1"/>
+<wire x1="17.78" y1="5.08" x2="24.13" y2="5.08" width="0" layer="19" extent="1-1"/>
 <wire x1="26.67" y1="15.24" x2="24.13" y2="5.08" width="0" layer="19" extent="1-1"/>
 </signal>
@@
 <contactref element="AMBIENT_TEMP_SENSOR" pad="2"/>
 <contactref element="B1" pad="A5"/>
-<contactref element="THROUGH_HOLE_AMBIENT_TEMP_SENSOR" pad="2"/>
-<wire x1="11.43" y1="80.01" x2="83.82" y2="85.09" width="0" layer="19" extent="1-1"/>
-<wire x1="52.07" y1="15.24" x2="11.43" y2="80.01" width="0" layer="19" extent="1-1"/>
+<wire x1="52.07" y1="15.24" x2="83.82" y2="85.09" width="0" layer="19" extent="1-1"/>
 </signal>
 <signal name="N$22">
@@
 <wire x1="85.09" y1="27.94" x2="60.96" y2="85.09" width="0" layer="19" extent="1-1"/>
 </signal>
+<signal name="N$26">
+</signal>
+<signal name="N$28">
+<contactref element="B1" pad="A6"/>
+<contactref element="T2" pad="2"/>
+<wire x1="-8.89" y1="-31.115" x2="54.61" y2="15.24" width="0" layer="19" extent="1-1"/>
+</signal>
 <signal name="N$25">
-<contactref element="THROUGH_HOLE_AMBIENT_TEMP_SENSOR" pad="1"/>
 <contactref element="JP11" pad="1"/>
-<wire x1="8.89" y1="80.01" x2="80.01" y2="2.54" width="0" layer="19" extent="1-1"/>
-</signal>
-<signal name="N$26">
+<contactref element="T2" pad="3"/>
+<wire x1="-10.16" y1="-33.02" x2="80.01" y2="2.54" width="0" layer="19" extent="1-1"/>
+</signal>
+<signal name="N$27">
+<contactref element="JP11" pad="2"/>
+</signal>
+<signal name="N$29">
+<contactref element="B1" pad="3.3V"/>
 </signal>
 </signals>

Commit message: Removed .DS_Store file and changed board schematics
Parts:
- added Q1, Q2: 2N5496, transistor-npn:TO220
- added R3, R4: 4.7K, rcl:0207/10
- added R5, R8: 5.3K, rcl:0207/10
- added R6, R7: 2K, rcl:0207/10
- renumbered AMBIENT_TEMP_SENSOR to DS18B20
Connections:
- net N$10 renamed EN_ACT2
- net N$22 renamed HW_SS
- net N$23 renamed CS_T1
- net N$5 renamed CS_T2
- net N$9 renamed EN_ACT1
- removed net 5V: 5V.1, B1.5V@0, JP1.2, JP10.1, JP2.2, JP3.2, JP4.2, JP5.2, JP6.2, JP7.2, JP8.1, JP9.1
- removed net N$19: TEMP1.4
- removed net N$2 (its old number): B1.51, MOSI.1, RF69.4, SDCARD.6, TRACKSOAR.3
- removed net N$24: B1.A5, DS18B20.2
- removed net N$27: JP11.2
- removed net N$28: B1.A6, T2.2
- removed net N$4: B1.52, RF69.5, SDCARD.4, SPI_CLK.1, TEMP.1, TEMP1.1, TRACKSOAR.5
- removed net N$6: B1.18, RF69.6
- new net 1NAME: B1.46
- new net AM_TEMP1: B1.34, R3.2, T2.2
- new net AM_TEMP2: B1.36, DS18B20.2, R4.2
- new net CS_RF: B1.18
- new net MISO: B1.50, MISO.1, RF69.3, SDCARD.5, TEMP.3, TEMP1.3, TRACKSOAR.5
- new net MOSI: B1.47, B1.51, MOSI.1, RF69.4, SDCARD.6, SDCARD.7, TRACKSOAR.4
- new net RF_CS: RF69.6
- new net SCK: B1.52, RF69.5, SDCARD.4, SPI_CLK.1, TEMP.1, TEMP1.1, TRACKSOAR.3
- new net VCC: 5V.1, B1.5V@0, JP1.2, JP10.1, JP11.2, JP2.2, JP3.2, JP4.2, JP5.2, JP6.2, JP7.2, JP8.1, JP9.1, R3.1, R4.1
- net GND: now also Q2.3, TEMP1.4; no longer ACTUATOR_2.3
- net N$1: now also Q2.1, R5.1, R6.2; no longer B1.47, SDCARD.7
- net N$3: now also ACTUATOR_2.3, Q2.2; no longer B1.50, MISO.1, RF69.3, SDCARD.5, TEMP.3, TEMP1.3, TRACKSOAR.4
Routing:
- net SCK: track 0.00 -> 232.2 mm, vias 0 -> 6
- net N$4: track 232.2 -> 0.00 mm, vias 6 -> 0
- net N$3: track 227.5 -> 0.00 mm, vias 1 -> 0
- net MISO: track 0.00 -> 227.5 mm, vias 0 -> 1
- net MOSI: track 0.00 -> 194.5 mm, vias 0 -> 6
- net N$2 (its old number): track 160.2 -> 0.00 mm, vias 3 -> 0
- net N$1: track 54.0 -> 0.00 mm, vias 3 -> 0
- net N$6: track 43.1 -> 0.00 mm, vias 1 -> 0
- net RF_CS: track 0.00 -> 41.8 mm, vias 0 -> 1
- net SDA: track 132.1 -> 116.9 mm
- net VCC: track 0.00 -> 14.5 mm
- net 5V: track 14.5 -> 0.00 mm
- net SCL: track 118.5 -> 108.0 mm
- net CS_T2: track 80.4 -> 75.0 mm

Commit message: finished schematic
Parts:
- removed JP8: (no value), jumper:JP1
- removed TEMP: (no value), con-lsta:FE06
- added JP12: (no value), jumper:JP1
- added TEMP2: (no value), con-lsta:FE06
- moved TEMP1 72.0 mm to (10.2, 38.1)
Connections:
- removed net 1NAME: B1.46
- removed net N$14: JP3.1, RF69.9
- removed net N$15: JP7.1, TEMP.6
- removed net N$18: JP8.2, TEMP1.6
- removed net RF_CS: RF69.6
- new net COM_ACT1: ACTUATOR_1.1, B1.2
- new net COM_ACT2: ACTUATOR_2.1, B1.3
- new net CS_SD: B1.47, SDCARD.7
- new net INT_RF: B1.18, RF69.4
- new net N$4: Q1.1, R7.1, R8.2
- new net N$5: ACTUATOR_1.3, Q1.2
- new net N$6: JP3.1, RF69.1
- new net RST_RF: B1.45, RF69.9
- net CS_RF: now also B1.44, RF69.8; no longer B1.18
- net CS_T1: now also TEMP2.5; no longer TEMP1.2
- net CS_T2: now also TEMP1.5; no longer TEMP.2
- net EN_ACT1: now also R7.2; no longer ACTUATOR_1.1, B1.2
- net EN_ACT2: now also R6.1; no longer ACTUATOR_2.1, B1.3
- net GND: now also Q1.3, R5.2, R8.1, RF69.2, TEMP1.3, TEMP2.3; no longer ACTUATOR_1.3, RF69.8, TEMP.4, TEMP1.4
- net MISO: now also RF69.6, TEMP1.4, TEMP2.4; no longer RF69.3, TEMP.3, TEMP1.3
- net MOSI: now also RF69.7; no longer B1.47, RF69.4, SDCARD.7
- net N$7: now also JP7.1, TEMP1.1; no longer B1.44, RF69.2
- net N$8: now also JP12.1, TEMP2.1; no longer B1.45, RF69.1
- net SCK: now also TEMP1.6, TEMP2.6; no longer TEMP.1, TEMP1.1
- net VCC: now also JP12.2; no longer JP8.1
Routing:
- net N$8: track 117.8 -> 0.00 mm, vias 1 -> 0
- net RST_RF: track 0.00 -> 116.0 mm, vias 0 -> 1
- net MOSI: track 194.5 -> 95.7 mm, vias 6 -> 1
- net N$7: track 92.9 -> 0.00 mm, vias 1 -> 0
- net CS_RF: track 0.00 -> 89.0 mm, vias 0 -> 1
- net CS_T2: track 75.0 -> 0.00 mm, vias 1 -> 0
- net SCK: track 232.2 -> 175.1 mm, vias 6 -> 4
- net CS_SD: track 0.00 -> 51.5 mm, vias 0 -> 3
- net INT_RF: track 0.00 -> 43.0 mm, vias 0 -> 2
- net RF_CS: track 41.8 -> 0.00 mm, vias 1 -> 0
- net MISO: track 227.5 -> 248.4 mm, vias 1 -> 2
- net GND: track 123.5 -> 117.7 mm

Commit message: placed and routed hab board
Parts:
- moved R8 238.0 mm to (54.6, 83.8), turned to 180 degrees
- moved TEMP2 235.7 mm to (92.7, 27.9), turned to 270 degrees
- moved R7 217.7 mm to (54.6, 74.9)
- moved R6 193.8 mm to (29.2, 74.9), turned to 180 degrees
- moved R5 188.1 mm to (29.2, 82.5)
- moved JP12 172.5 mm to (31.8, 3.81), turned to 180 degrees
- moved Q1 153.5 mm to (67.3, 82.5), turned to 180 degrees
- moved Q2 151.9 mm to (41.9, 82.5), turned to 180 degrees
- moved R4 119.6 mm to (44.5, -1.27)
- moved R3 114.5 mm to (44.5, 3.81)
- moved DS18B20 92.8 mm to (57.1, -3.81)
- moved JP11 86.4 mm to (-6.35, 3.81)
- moved TRACKSOAR 85.3 mm to (80.0, -6.35)
- moved TEMP1 83.3 mm to (92.7, 49.5), turned to 270 degrees
- moved MISO 78.8 mm to (78.7, 2.54)
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Routing:
- net N$7: track 0.00 -> 151.3 mm
- net N$17: track 0.00 -> 129.7 mm
- net GND: track 117.7 -> 0.00 mm, vias 1 -> 0
- net N$16: track 0.00 -> 117.5 mm, vias 0 -> 1
- net N$6: track 0.00 -> 115.4 mm, vias 0 -> 2
- net SCL: track 108.0 -> 213.9 mm, vias 5 -> 3
- net N$20: track 0.00 -> 104.1 mm
- net N$8: track 0.00 -> 87.1 mm, vias 0 -> 2
- net N$11: track 0.00 -> 86.8 mm, vias 0 -> 1
- net MOSI: track 95.7 -> 179.2 mm, vias 1 -> 3
- net AM_TEMP2: track 0.00 -> 78.3 mm
- net MISO: track 248.4 -> 171.5 mm, vias 2 -> 0
- net SDA: track 116.9 -> 192.9 mm, vias 3 -> 2
- net AM_TEMP1: track 0.00 -> 73.6 mm
- net N$2: track 0.00 -> 70.4 mm, vias 0 -> 1
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- added copper zone on layer 16, net GND
Other:
- board size 120.3 x 101.6 mm -> 127.1 x 101.7 mm
