File: HAB3_pcb/integrated-board/paxtanLaker/IMUqfn/ICM20689/ICM20689.sch (KiCad schematic (older format))
At the start: 7 parts, among them J1 Conn_01x03_Male, J2 Conn_01x06_Male, U1 ICM-20689

Commit message: made fixes to new imu
Parts:
- U1: symbol ICM-20689:ICM-20689 -> ICM20689-rescue:ICM-20689-ICM-20689
Changed lines of the file:
@@
 EESchema Schematic File Version 4
+LIBS:ICM20689-cache
 EELAYER 26 0
 EELAYER END
@@
 $EndDescr
 $Comp
-L ICM-20689:ICM-20689 U1
+L ICM20689-rescue:ICM-20689-ICM-20689 U1
 U 1 1 5BD15253
 P 5850 4050
