File: HAB3_pcb/makena-thermocoupler/Hab_thermocoupler.sch (KiCad schematic (older format))
At the start: 11 parts, among them J1 Conn_01x02_Male, J2 Conn_01x06_Female, U1 MAX31855

Commit message: changed diodes to be SOD 123 and updated footprint
Parts:
- D1, D2: footprint Diode_SMD:D_0402_1005Metric -> Diode_SMD:D_SOD-123
Changed lines of the file:
@@
 F 0 "D2" H 6650 3684 50  0000 C CNN
 F 1 "1N4148" H 6650 3775 50  0000 C CNN
-F 2 "Diode_SMD:D_0402_1005Metric" H 6650 3900 50  0001 C CNN
+F 2 "Diode_SMD:D_SOD-123" H 6650 3900 50  0001 C CNN
 F 3 "~" H 6650 3900 50  0001 C CNN
 	1    6650 3900
@@
 F 0 "D1" H 6650 3484 50  0000 C CNN
 F 1 "1N4148" H 6650 3575 50  0000 C CNN
-F 2 "Diode_SMD:D_0402_1005Metric" H 6650 3700 50  0001 C CNN
+F 2 "Diode_SMD:D_SOD-123" H 6650 3700 50  0001 C CNN
 F 3 "~" H 6650 3700 50  0001 C CNN
 	1    6650 3700

Commit message: changed schematic and footprint following design review
Parts:
- removed D1, D2: 1N4148, Diode_SMD:D_SOD-123, symbol Device:D
- removed J2: Conn_01x06_Female, Connector_PinSocket_2.54mm:PinSocket_1x06_P2.54mm_Vertical, symbol Connector:Conn_01x06_Female
- removed R1, R2: 10k, Resistor_SMD:R_0402_1005Metric, symbol Device:R
- added J2: Conn_01x05_Female, Connector_PinSocket_2.54mm:PinSocket_1x05_P2.54mm_Vertical, symbol Connector:Conn_01x05_Female
- C1, C2: footprint Capacitor_SMD:C_0402_1005Metric -> Capacitor_SMD:C_0603_1608Metric
- L1, L2: footprint Inductor_SMD:L_0402_1005Metric -> Inductor_SMD:L_0603_1608Metric
Connections:
- net labels removed: +5V
- wire segments 46 -> 37
Changed lines of the file:
@@
 F 0 "C1" H 4515 3746 50  0000 L CNN
 F 1 ".01 uF" H 4515 3655 50  0000 L CNN
-F 2 "Capacitor_SMD:C_0402_1005Metric" H 4438 3550 50  0001 C CNN
+F 2 "Capacitor_SMD:C_0603_1608Metric" H 4438 3550 50  0001 C CNN
 F 3 "~" H 4400 3700 50  0001 C CNN
 	1    4400 3700
@@
 	4650 3800 5100 3800
 $Comp
-L Device:R R1
-U 1 1 5BB5A697
-P 6250 3500
-F 0 "R1" H 6320 3546 50  0000 L CNN
-F 1 "10k" H 6320 3455 50  0000 L CNN
-F 2 "Resistor_SMD:R_0402_1005Metric" V 6180 3500 50  0001 C CNN
-F 3 "~" H 6250 3500 50  0001 C CNN
-	1    6250 3500
-	1    0    0    -1
-$EndComp
-$Comp
 L Device:Ferrite_Bead L1
 U 1 1 5BB5A7BF
@@
 F 0 "L1" V 3726 3550 50  0000 C CNN
 F 1 "Ferrite_Bead" V 3817 3550 50  0000 C CNN
-F 2 "Inductor_SMD:L_0402_1005Metric" V 3930 3550 50  0001 C CNN
+F 2 "Inductor_SMD:L_0603_1608Metric" V 3930 3550 50  0001 C CNN
 F 3 "~" H 4000 3550 50  0001 C CNN
 	1    4000 3550
@@
 F 0 "L2" V 3726 3850 50  0000 C CNN
 F 1 "Ferrite_Bead" V 3817 3850 50  0000 C CNN
-F 2 "Inductor_SMD:L_0402_1005Metric" V 3930 3850 50  0001 C CNN
+F 2 "Inductor_SMD:L_0603_1608Metric" V 3930 3850 50  0001 C CNN
 F 3 "~" H 4000 3850 50  0001 C CNN
 	1    4000 3850
@@
 	3500 3850 3850 3850
 $Comp
-L Device:D D2
-U 1 1 5BB5B70F
-P 6650 3900
-F 0 "D2" H 6650 3684 50  0000 C CNN
-F 1 "1N4148" H 6650 3775 50  0000 C CNN
-F 2 "Diode_SMD:D_SOD-123" H 6650 3900 50  0001 C CNN
-F 3 "~" H 6650 3900 50  0001 C CNN
-	1    6650 3900
-	-1   0    0    1
-$EndComp
-$Comp
-L Device:D D1
-U 1 1 5BB5B7A9
-P 6650 3700
-F 0 "D1" H 6650 3484 50  0000 C CNN
-F 1 "1N4148" H 6650 3575 50  0000 C CNN
-F 2 "Diode_SMD:D_SOD-123" H 6650 3700 50  0001 C CNN
-F 3 "~" H 6650 3700 50  0001 C CNN
-	1    6650 3700
-	-1   0    0    1
-$EndComp
-$Comp
-L Device:R R2
-U 1 1 5BB5B92E
-P 6250 4150
-F 0 "R2" H 6320 4196 50  0000 L CNN
-F 1 "10k" H 6320 4105 50  0000 L CNN
-F 2 "Resistor_SMD:R_0402_1005Metric" V 6180 4150 50  0001 C CNN
-F 3 "~" H 6250 4150 50  0001 C CNN
-	1    6250 4150
-	1    0    0    -1
-$EndComp
-Wire Wire Line
-	5900 3900 6250 3900
-Wire Wire Line
-	6250 4000 6250 3900
-Connection ~ 6250 3900
-Wire Wire Line
-	6250 3900 6500 3900
-Wire Wire Line
-	5900 3700 6250 3700
-Wire Wire Line
-	6250 3700 6250 3650
-Connection ~ 6250 3700
-Wire Wire Line
-	6250 3700 6500 3700
-Wire Wire Line
-	5900 3500 6000 3500
-Wire Wire Line
-	7450 3400 7450 4000
-Wire Wire Line
-	7450 4000 7700 4000
-Wire Wire Line
-	6700 3400 7450 3400
-$Comp
-L Connector:Conn_01x06_Female J2
-U 1 1 5BB5C524
-P 7900 3900
-F 0 "J2" H 7927 3876 50  0000 L CNN
-F 1 "Conn_01x06_Female" H 7900 3450 50  0000 L CNN
-F 2 "Connector_PinSocket_2.54mm:PinSocket_1x06_P2.54mm_Vertical" H 7900 3900 50  0001 C CNN
-F 3 "~" H 7900 3900 50  0001 C CNN
-	1    7900 3900
-	1    0    0    -1
-$EndComp
-$Comp
-L power:+5V #PWR05
-U 1 1 5BB5C5B8
-P 7700 3700
-F 0 "#PWR05" H 7700 3550 50  0001 C CNN
-F 1 "+5V" H 7715 3873 50  0000 C CNN
-F 2 "" H 7700 3700 50  0001 C CNN
-F 3 "" H 7700 3700 50  0001 C CNN
-	1    7700 3700
-	1    0    0    -1
-$EndComp
-$Comp
 L power:GND #PWR07
 U 1 1 5BB5C6BA
-P 8250 3900
-F 0 "#PWR07" H 8250 3650 50  0001 C CNN
-F 1 "GND" V 8255 3772 50  0000 R CNN
-F 2 "" H 8250 3900 50  0001 C CNN
-F 3 "" H 8250 3900 50  0001 C CNN
-	1    8250 3900
+P 7900 3900
+F 0 "#PWR07" H 7900 3650 50  0001 C CNN
+F 1 "GND" V 7905 3772 50  0000 R CNN
+F 2 "" H 7900 3900 50  0001 C CNN
+F 3 "" H 7900 3900 50  0001 C CNN
+	1    7900 3900
 	0    -1   -1   0
 $EndComp
-Wire Wire Line
-	7700 3900 8250 3900
-Wire Wire Line
-	7700 4100 6800 4100
-Wire Wire Line
-	6800 4100 6800 3900
-Wire Wire Line
-	6800 3700 7300 3700
-Wire Wire Line
-	7300 3700 7300 4200
-Wire Wire Line
-	7300 4200 7700 4200
 $Comp
 L Device:C C2
@@
 F 0 "C2" H 5700 2950 50  0000 L CNN
 F 1 "0.1 uF" H 5500 2850 50  0000 L CNN
-F 2 "Capacitor_SMD:C_0402_1005Metric" H 5638 2800 50  0001 C CNN
+F 2 "Capacitor_SMD:C_0603_1608Metric" H 5638 2800 50  0001 C CNN
 F 3 "~" H 5600 2950 50  0001 C CNN
 	1    5600 2950
@@
 $EndComp
 Wire Wire Line
-	7700 3800 7550 3800
-Wire Wire Line
-	7550 3800 7550 3200
-Wire Wire Line
 	5100 2950 5450 2950
 Wire Wire Line
 	5100 2950 5100 3400
-Wire Wire Line
-	5750 2950 7550 2950
-Wire Wire Line
-	6000 3500 6000 3000
-Wire Wire Line
-	6000 3000 6700 3000
-Wire Wire Line
-	6700 3000 6700 3400
-Wire Wire Line
-	6250 3350 6250 3200
-Wire Wire Line
-	6250 3200 7550 3200
-Connection ~ 7550 3200
-Wire Wire Line
-	7550 3200 7550 2950
-Wire Wire Line
-	6250 4300 6250 4600
-Wire Wire Line
-	6250 4600 7550 4600
-Wire Wire Line
-	7550 4600 7550 3800
-Connection ~ 7550 3800
 Wire Wire Line
 	5100 4000 5100 4750
@@
 Wire Wire Line
 	7650 3900 7700 3900
-Connection ~ 7700 3900
 $Comp
 L power:+3V3 #PWR0101
@@
 	0    -1   -1   0
 $EndComp
+Wire Wire Line
+	5100 2950 5100 2700
+Wire Wire Line
+	5100 2700 7500 2700
+Wire Wire Line
+	7500 2700 7500 3800
+Connection ~ 5100 2950
+Wire Wire Line
+	7400 2950 7400 3900
+Wire Wire Line
+	7400 3900 7650 3900
+Connection ~ 7650 3900
+Wire Wire Line
+	5750 2950 7400 2950
+Wire Wire Line
+	5900 4200 5900 3900
+Wire Wire Line
+	5900 3700 6000 3700
+Wire Wire Line
+	7700 4000 6100 4000
+Wire Wire Line
+	6100 4000 6100 3500
+Wire Wire Line
+	6100 3500 5900 3500
+$Comp
+L Connector:Conn_01x05_Female J2
+U 1 1 5BD6D44D
+P 7900 4000
+F 0 "J2" H 7800 3700 50  0000 L CNN
+F 1 "Conn_01x05_Female" H 7850 3600 50  0000 L CNN
+F 2 "Connector_PinSocket_2.54mm:PinSocket_1x05_P2.54mm_Vertical" H 7900 4000 50  0001 C CNN
+F 3 "~" H 7900 4000 50  0001 C CNN
+	1    7900 4000
+	1    0    0    -1
+$EndComp
+Wire Wire Line
+	7500 3800 7700 3800
+Connection ~ 7700 3800
+Wire Wire Line
+	7700 3800 7750 3800
+Wire Wire Line
+	5900 4200 7450 4200
+Wire Wire Line
+	7450 4200 7450 4100
+Wire Wire Line
+	7450 4100 7700 4100
+Wire Wire Line
+	6000 4350 7700 4350
+Wire Wire Line
+	7700 4350 7700 4200
+Wire Wire Line
+	6000 3700 6000 4350
 $EndSCHEMATC
