File: HAB3_pcb/riley/AltimeterPCB/AltimeterPCB.sch (KiCad schematic (older format))
At the start: 4 parts, among them J1 Conn_01x04_Female, J2 Conn_02x01, U1 MS560702BA03-00

Commit message: changed fonts to be thicker, 0402 -> 0603_hand_solder
Parts:
- C1: footprint Capacitor_SMD:C_0402_1005Metric -> Capacitor_SMD:C_0603_1608Metric_Pad1.05x0.95mm_HandSolder
Changed lines of the file:
@@
 F 0 "C1" H 3778 3146 50  0000 L CNN
 F 1 "100nF" H 3778 3055 50  0000 L CNN
-F 2 "Capacitor_SMD:C_0402_1005Metric" H 3600 3100 50  0001 C CNN
+F 2 "Capacitor_SMD:C_0603_1608Metric_Pad1.05x0.95mm_HandSolder" H 3600 3100 50  0001 C CNN
 F 3 "" H 3600 3100 50  0001 C CNN
 	1    3600 3100
