File: HAB3_pcb/integrated-board/tim-integrated-board/integrated-board/integrated-board.kicad_pcb (KiCad board)
At the start: 4 copper layers, 134.4 x 98.9 mm, 122 parts, among them IC1 RTC_PCF8523T, J1 Conn_01x02_Male, J1 Conn_01x03_Male, J1 Conn_01x09_Female, J1 Conn_ARM_JTAG_SWD_20, J10 Conn_01x02_Male, J12 Conn_01x03_Male, J13 Conn_01x04_Male, J14 Conn_01x05_Male, J15 Conn_01x08_Male, J2 Conn_01x02_Female, J2 Conn_01x06_Female, J2 Conn_01x06_Male, J2 Micro_SD_Card_Det, J3 Conn_01x16_Male, J4 Conn_01x16_Male, J5 Conn_01x16_Male, J6 Conn_01x02_Male, J7 Conn_01x02_Male, J8 Conn_01x02_Male, J9 Conn_01x11_Male, Q1 32.768KHz, SW1 SW_DPST_x2, U1 FGPMMOPA6H, U1 ICM-20689, U1 LSM9DS0, U1 MAX31855, U1 MS560702BA03-00, U1 STM32F401RET6, U2 TPS564208, U3 TPS564208, Y1 32.768MHz

Commit message: made fixes to new imu
Parts:
- moved C3 14.3 mm to (93.4, 45.9), turned to 180 degrees
- moved C4 10.8 mm to (93.4, 47.6), turned to 180 degrees
- moved C1 10.8 mm to (89.1, 51.8), turned to 90 degrees
- moved C2 9.99 mm to (86.9, 50.2), turned to 270 degrees
Routing:
- net VDD: track 47.9 -> 20.7 mm, vias 4 -> 2
- net GND: track 196.9 -> 220.2 mm, vias 50 -> 52
- net VDDIO: track 23.1 -> 11.5 mm
- net Net-(C1-Pad2): track 97.9 -> 86.4 mm, vias 3 -> 1
- net SDA: track 45.2 -> 38.4 mm
- net nCS: track 34.9 -> 28.1 mm
- net SCL: track 40.5 -> 33.8 mm
- net AD0: track 20.7 -> 23.2 mm, vias 1 -> 0

Commit message: fixed power on integrated board
Parts:
- removed the B1 at (83.4, 98.9)
- removed the C1 at (84.5, 122.8)
- removed the C1 at (85.5, 89.6)
- removed the D1 at (103.6, 126.6)
- removed the D1 at (99.6, 89.7)
- removed the D2 at (103.6, 121.6)
- removed the D2 at (97.5, 109.2)
- removed FID1, FID2: FIDUCIAL, Adafruit Ultimate GPS:FIDUCIAL_1MM
- removed J15: Conn_01x08_Male, Pin_Headers:Pin_Header_Straight_1x08_Pitch2.54mm
- removed the J2 at (108.7, 113.9)
- removed LED1: RED, Adafruit Ultimate GPS:CHIPLED_0805
- removed the R1 at (98.5, 126.1)
- removed the R1 at (92.5, 109.5)
- removed U$16: , Adafruit Ultimate GPS:PCBFEAT-REV-040
- removed U$20: U.FL, Adafruit Ultimate GPS:U.FL
- removed the U$8 at (78.7, 109.1)
- removed the U$9 at (78.7, 88.7)
- removed the U1 at (90.9, 122.8)
- removed the U1 at (92.9, 99.4)
- added @HOLE0: , , F.Cu at (123.4, 90.8)
- added @HOLE1: , , F.Cu at (124.7, 90.8)
- added @HOLE10: , , F.Cu at (166.0, 100.6)
- added @HOLE11: , , F.Cu at (166.0, 99.3)
- added @HOLE12: , , F.Cu at (166.0, 98.1)
- added @HOLE13: , , F.Cu at (166.0, 96.8)
- added @HOLE2: , , F.Cu at (125.9, 90.8)
- added @HOLE3: , , F.Cu at (127.2, 90.8)
- added @HOLE4: , , F.Cu at (128.5, 90.8)
- added @HOLE5: , , F.Cu at (129.8, 90.8)
- added @HOLE6: , , F.Cu at (131.0, 90.8)
- added @HOLE7: , , F.Cu at (166.0, 104.4)
- added @HOLE8: , , F.Cu at (166.0, 103.2)
- added @HOLE9: , , F.Cu at (166.0, 101.9)
- added C1: .1uf, Tracksoar v2 :0402-CAP, F.Cu at (164.2, 91.7)
- added C10: .1uf, Tracksoar v2 :0402-CAP, B.Cu at (231.9, 69.4)
- added C11: .1uf, Tracksoar v2 :0402-CAP, F.Cu at (155.9, 92.3)
- added C12: 1uf, Tracksoar v2 :0402-CAP, B.Cu at (134.2, 103.6)
- added C13: .1uf, Tracksoar v2 :0402-CAP, F.Cu at (130.5, 93.3)
- added C14: .1uf, Tracksoar v2 :0402-CAP, F.Cu at (151.0, 101.0)
- added C15: 10uF, Tracksoar v2 :0603, F.Cu at (150.4, 97.1)
- added C16: 10uF, Tracksoar v2 :0603, F.Cu at (153.0, 94.2)
- added C17: .1uf, Tracksoar v2 :0402-CAP, F.Cu at (163.4, 101.6)
- added C3: GPS BACKUP, Tracksoar v2 :DSK-3R3H204T614-H2L, F.Cu at (159.3, 98.4)
- added C4: .1uf, Tracksoar v2 :0402-CAP, B.Cu at (146.6, 102.0)
- added C5: 1uf, Tracksoar v2 :0402-CAP, B.Cu at (135.4, 96.8)
- added C6: .1uf, Tracksoar v2 :0402-CAP, B.Cu at (134.3, 106.4)
- added C7: 22uf, Tracksoar v2 :0805, F.Cu at (143.4, 96.7)
- added C8: 10uf, Tracksoar v2 :0805, F.Cu at (137.6, 96.1)
- added C9: .1uf, Tracksoar v2 :0402-CAP, B.Cu at (131.4, 94.7)
- added D1: MBR120VLSFT1, Tracksoar v2 :SOD123, F.Cu at (133.3, 100.3)
- added D2: SD101CW, Tracksoar v2 :SOD-123, F.Cu at (164.6, 95.9)
- added F1: PTC0603, Tracksoar v2 :0603, B.Cu at (131.4, 96.3)
- added FRAME1: FRAME-LETTER, Tracksoar v2 :CREATIVE_COMMONS, F.Cu at (132.0, 123.1)
- added FTDI1: 1X8, Tracksoar v2 :1X8, F.Cu at (139.6, 91.8)
- added GPS-ANT1: 1.575GHz, Tracksoar v2 :ANT-GPS-2X7MM, B.Cu at (167.9, 108.4)
- added GPSLOCK1: LEDCHIP-LED0603, Tracksoar v2 :CHIP-LED0603, B.Cu at (161.8, 91.6)
- added H1: MOUNT-HOLE2.8, Tracksoar v2 :2,8, F.Cu at (127.2, 86.2)
- added H2: MOUNT-HOLE2.8, Tracksoar v2 :2,8, F.Cu at (170.6, 100.7)
- added IC1: BME280, Tracksoar v2 :BME280, F.Cu at (149.3, 102.6)
- added J$1: SMA_EDGE, Tracksoar v2 :SMA-EDGE, B.Cu at (205.2, 71.9)
- added J20: Conn_01x03_Male, Pin_Headers:Pin_Header_Straight_1x03_Pitch2.54mm, F.Cu at (434.2, 44.0)
- added J21: Conn_01x05_Male, Pin_Headers:Pin_Header_Straight_1x05_Pitch2.54mm, F.Cu at (430.6, 44.0)
- added LT3426: LT3426, Tracksoar v2 :SOT23-6, F.Cu at (141.2, 100.2)
- added PTT1: LEDCHIP-LED0603, Tracksoar v2 :CHIP-LED0603, B.Cu at (139.4, 107.1)
- added R1: 1k, Tracksoar v2 :R0402, B.Cu at (159.0, 91.6)
- added R10: 30.9k, Tracksoar v2 :R0402, F.Cu at (144.7, 100.7)
- added R11: 22ohm, Tracksoar v2 :R0402, F.Cu at (131.3, 96.9)
- added R12: 10k, Tracksoar v2 :R0402, B.Cu at (151.2, 104.6)
- added R13: 10k, Tracksoar v2 :R0402, B.Cu at (136.1, 104.7)
- added R14: 10k, Tracksoar v2 :R0402, B.Cu at (152.3, 99.0)
- added R15: 4.7k, Tracksoar v2 :R0402, B.Cu at (151.0, 99.0)
- added R16: 10k, Tracksoar v2 :R0402, B.Cu at (147.2, 99.2)
- added R17: 330, Tracksoar v2 :R0402, F.Cu at (164.6, 100.2)
- added R4: 22ohm, Tracksoar v2 :R0402, B.Cu at (131.3, 98.2)
- added R5: 10k, Tracksoar v2 :R0402, B.Cu at (135.0, 94.6)
- added R6: 1k, Tracksoar v2 :R0402, B.Cu at (144.1, 106.3)
- added R7: 4.7k, Tracksoar v2 :R0402, B.Cu at (147.6, 95.4)
- added R8: 1m, Tracksoar v2 :R0402, F.Cu at (141.0, 97.1)
- added R9: 95.3k, Tracksoar v2 :R0402, F.Cu at (143.4, 100.7)
- added REF**: Pin_Header_Straight_1x03_Pitch2.54mm, Pin_Headers:Pin_Header_Straight_1x03_Pitch2.54mm, F.Cu at (218.8, 72.3)
- added REF**: Pin_Header_Straight_1x04_Pitch2.54mm, Pin_Headers:Pin_Header_Straight_1x04_Pitch2.54mm, F.Cu at (240.2, 72.1)
- added U$1: UBLOX_MAX, Tracksoar v2 :UBLOX_MAX, B.Cu at (160.3, 99.3)
- added U$2: RADIOMETRIX-HX1, Tracksoar v2 :RADIOMETRIX-HX1, F.Cu at (224.9, 61.8)
- added U$3: 1X6, Tracksoar v2 :1X6, F.Cu at (140.4, 108.8)
- added U$4: ATMEGA32U4, Tracksoar v2 :QFN-44-NOPAD, B.Cu at (140.4, 100.5)
- added U$5: PAM2305, Tracksoar v2 :DBV_R-PDSO-G5, F.Cu at (150.2, 94.6)
- added U$6: 4.7uH, Tracksoar v2 :RESC0805_N, F.Cu at (147.3, 94.8)
- added U$7: INDUCTOR_0402_N, Tracksoar v2 :RESC0402_N, B.Cu at (131.0, 104.1)
- added Y1: 16MHZ, Tracksoar v2 :RESONATOR-SMD, B.Cu at (144.6, 94.7)
- C1: footprint Capacitor_SMD:C_0402_1005Metric -> Capacitors_SMD:C_0603_HandSoldering
- C2: value 0.1 uF -> .1uf; footprint Capacitor_SMD:C_0402_1005Metric -> Tracksoar v2 :0402-CAP; moved to B.Cu
- J1: value Conn_01x02_Male -> battery; footprint Connector_PinHeader_2.54mm:PinHeader_1x02_P2.54mm_Vertical -> Tracksoar v2 :JST-2-PTH; moved to B.Cu
- JP1: value HEADER-1X970MIL -> USB-MICROB; footprint Adafruit Ultimate GPS:1X09_ROUND_70 -> Tracksoar v2 :USB-MICROB
- L1: value Ferrite_Bead -> BLM15H; footprint Inductor_SMD:L_0402_1005Metric -> Tracksoar v2 :0402
- L2: value Ferrite_Bead -> 2.2uh; footprint Inductor_SMD:L_0402_1005Metric -> Tracksoar v2 :L1812
- R2: value 10k -> 4.7k; footprint Resistor_SMD:R_0402_1005Metric -> Tracksoar v2 :R0402
- R3: value 10K -> 4.7k; footprint Adafruit Ultimate GPS:0805-NO -> Tracksoar v2 :R0402; moved to B.Cu
- moved C1 237.4 mm to (430.8, 128.9)
- moved 100nF2 237.3 mm to (383.2, 64.6)
- moved 100nF3 237.3 mm to (387.0, 86.9)
- moved 100nF4 237.3 mm to (394.7, 87.1)
- moved 1uF2 237.3 mm to (384.6, 64.6)
- moved C2 237.3 mm to (360.4, 126.9)
- moved J10 237.3 mm to (431.0, 89.5)
- moved J2 237.3 mm to (341.6, 42.2)
- moved JP2 237.3 mm to (368.0, 120.0)
- moved R3 237.3 mm to (364.2, 126.9)
- moved R7 237.3 mm to (440.9, 100.3)
- moved U$8 237.3 mm to (312.4, 82.7)
- moved U$9 237.3 mm to (312.5, 38.7)
- moved U3 237.3 mm to (435.1, 99.5)
- moved 0k1 237.3 mm to (376.9, 72.7)
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Connections:
- C2 pad 1: Net-(C2-Pad1) -> GND
- C2 pad 2: Net-(C2-Pad2) -> VCC
- J1 pad 1: Net-(J1-Pad1) -> GND
- J1 pad 2: Net-(J1-Pad2) -> /VIN
- L1 pad 1: Net-(C1-Pad1) -> Net-(C7-Pad1)
- L1 pad 2: Net-(J1-Pad1) -> VCC
- L2 pad 1: Net-(C1-Pad2) -> /VIN
- L2 pad 2: Net-(J1-Pad2) -> Net-(D1-PadA)
- R2 pad 1: Net-(D2-Pad2) -> /3V
- R2 pad 2: Net-(C2-Pad2) -> Net-(IC1-Pad2)
- R3 pad 1: 3.3V -> /3V
- R3 pad 2: /RX_3V -> /SDA
Routing:
- net Net-(C16-Pad1): track 85.1 -> 24.1 mm, vias 3 -> 4
- net 3.3V: track 55.7 -> 0.00 mm, vias 3 -> 0
- net VCC: track 9.77 -> 59.2 mm, vias 2 -> 5
- net Net-(J2-Pad4): track 58.0 -> 11.9 mm
- net GND: track 220.2 -> 262.6 mm, vias 52 -> 47
- net Net-(B1-Pad+$1): track 41.3 -> 0.00 mm, vias 1 -> 0
- net /3V: track 0.00 -> 36.0 mm, vias 0 -> 1
- net /SCL: track 3.72 -> 34.3 mm, vias 0 -> 1
- net /FIX: track 30.0 -> 0.00 mm, vias 2 -> 0
- net /1PPS: track 26.4 -> 0.00 mm, vias 1 -> 0
- net Net-(C1-Pad1): track 109.4 -> 84.0 mm
- net /SDA: track 4.57 -> 28.3 mm, vias 0 -> 1
- net /VIN: track 0.00 -> 22.3 mm
- net Net-(C17-Pad1): track 10.4 -> 30.9 mm, vias 2 -> 6
- net Net-(C2-Pad2): track 18.4 -> 0.00 mm, vias 1 -> 0
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- added copper zone on Route15, net +3V3
- added copper zone on F.Cu, net /3V
- added copper zone on B.Cu, net /RFGND
- added copper zone on F.Cu, net /RFGND
- added copper zone on Route2, net /RFGND
- added copper zone on F.Cu, net /VIN
- added copper zone on Route2, net GND
- added copper zone on F.Cu, net Net-(C16-Pad1)
- added copper zone on B.Cu, net Net-(C17-Pad1)
- added copper zone on B.Cu, net Net-(C20-Pad1)
- added copper zone on F.Cu, net Net-(C7-Pad1)
- added copper zone on F.Cu, net Net-(D1-PadA)
- added copper zone on F.Cu, net Net-(LT3426-Pad3)
- added copper zone on F.Cu, net Net-(LT3426-Pad4)
- added copper zone on F.Cu, net VCC
- removed copper zone on In2.Cu, net +3V3
- removed copper zone on In1.Cu, net GND
Other:
- board size 134.4 x 98.9 mm -> 322.1 x 98.9 mm
- net class Default: clearance 0.2 -> 0.127; trace_width 0.25 -> 0.6
- rule trace_clearance: 0.2 -> 0.127
- rule trace_min: 0.2 -> 0.1524
- board text added: "!RESET"
- board text added: "+"
- board text added: "3V"
- board text added: "<3 Swiss"
- board text added: "A0"
- board text added: "A1"
- board text added: "D8"
- board text added: "D9"
- board text added: "I2C"
- board text added: "MISO"
- board text added: "MOSI"
- board text added: "SCK"
- board text added: "SPI"
- board text added: "SS"
- board text added: "Tracksoar v2"
- board text removed: "3.3V"
- board text removed: "EN"
- board text removed: "FIX"
- board text removed: "Logic: 5V Tolerant"
- board text removed: "PPS"
- board text removed: "RTC Batt: CR1220"
- board text removed: "Red-"
- board text removed: "VBAT"
- board text removed: "VIN: 3.3-5V"
- board text removed: "Yellow+"
- board text removed: "adafruit!"
