File: HABIV/old_board_submodules/altimeter/AltimeterPCB.kicad_pcb (KiCad board)
At the start: 4 copper layers, 7 parts, among them U7 MS560702BA03-00

Commit message: finish submodules and combine
Changed lines of the file:
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@@
     (at 126.905 103.515)
     (attr smd)
-    (fp_text reference U7 (at -0.105 4.485) (layer F.SilkS)
+    (fp_text reference U7 (at 3.845 0.135) (layer F.SilkS)
       (effects (font (size 1.5 1.5) (thickness 0.375)))
     )
-    (fp_text value MS560702BA03-00 (at 10.695 0.385) (layer F.SilkS)
+    (fp_text value MS560702BA03-00 (at 6.045 3.535) (layer F.SilkS)
       (effects (font (size 1 1) (thickness 0.25)))
     )
@@
     (tags capacitor)
     (attr smd)
-    (fp_text reference C10 (at 2.6125 -0.05) (layer F.SilkS)
+    (fp_text reference C10 (at 2.4125 0) (layer F.SilkS)
       (effects (font (size 1 1) (thickness 0.15)))
     )
@@
       (effects (font (size 1 1) (thickness 0.15)))
     )
-    (fp_text value 0 (at 1.2875 -1.8 90) (layer F.Fab)
+    (fp_text value 0 (at -0.0125 -0.05 90) (layer F.Fab)
       (effects (font (size 1 1) (thickness 0.15)))
     )
@@
       (effects (font (size 1 1) (thickness 0.15)))
     )
-    (fp_text value 0 (at -2.6625 4.25 90) (layer F.Fab)
+    (fp_text value 0 (at -0.0125 0.05 90) (layer F.Fab)
       (effects (font (size 1 1) (thickness 0.15)))
     )
@@
       (effects (font (size 1 1) (thickness 0.15)))
     )
-    (fp_text value 0 (at -2.5625 0.1 90) (layer F.Fab)
+    (fp_text value 0 (at -0.1125 0.05 90) (layer F.Fab)
       (effects (font (size 1 1) (thickness 0.15)))
     )
@@
       (effects (font (size 1 1) (thickness 0.15)))
     )
-    (fp_text value 0 (at 0.3125 7.95 270) (layer F.Fab)
+    (fp_text value 0 (at -0.0375 0.1 270) (layer F.Fab)
       (effects (font (size 1 1) (thickness 0.15)))
     )
@@
       (effects (font (size 1 1) (thickness 0.15)))
     )
-    (fp_text value 0 (at -2.4625 -0.1) (layer F.Fab)
-      (effects (font (size 1 1) (thickness 0.15)))
-    )
+    (fp_text value 0 (at -0.0125 -0.05) (layer F.Fab)
+      (effects (font (size 1 1) (thickness 0.15)))
+    )
