File: HABIV/old_board_submodules/real_time_clock/real_time_clock.kicad_pcb (KiCad board)
At the start: 4 copper layers, 11 parts, among them IC1 RTC_PCF8523T, Q1 32.768KHz

Commit message: finish submodules and combine
Routing:
- net Net-(B2-Pad2): track 33.4 -> 21.5 mm, vias 0 -> 2
- net GND: track 23.7 -> 22.9 mm
Changed lines of the file:
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@@
     (thickness 1.6)
     (drawings 1)
-    (tracks 76)
+    (tracks 72)
     (zones 0)
     (modules 11)
@@
     (effects (font (size 1.5 1.5) (thickness 0.15)))
   )
-  (via (at 133.45 114.35) (size 0.8) (drill 0.4) (layers F.Cu B.Cu) (net 8))
-  (via (at 133.4 109.7) (size 0.8) (drill 0.4) (layers F.Cu B.Cu) (net 8))
   (segment (start 120.07 100.33) (end 120.07 112.45) (width 0.25) (layer F.Cu) (net 1) (status 10))
-  (segment (start 120.07 112.45) (end 121.92 114.3) (width 0.25) (layer F.Cu) (net 1) (status 20))
   (segment (start 122.34 114.3) (end 121.92 114.3) (width 0.25) (layer F.Cu) (net 1) (status 30))
   (segment (start 123.655 114.3) (end 122.34 114.3) (width 0.25) (layer F.Cu) (net 1) (status 20))
@@
   (segment (start 125.64 112.94) (end 127 114.3) (width 0.25) (layer F.Cu) (net 1) (status 20))
   (segment (start 125.64 111.76) (end 125.64 112.94) (width 0.25) (layer F.Cu) (net 1) (status 10))
-  (segment (start 121.5 114.3) (end 121.27499 114.52501) (width 0.25) (layer F.Cu) (net 1) (status 10))
-  (segment (start 121.92 114.3) (end 121.5 114.3) (width 0.25) (layer F.Cu) (net 1) (status 30))
+  (segment (start 120.07 112.45) (end 121.92 114.3) (width 0.25) (layer F.Cu) (net 1) (status 20))
   (via (at 132.4 108) (size 0.8) (drill 0.4) (layers F.Cu B.Cu) (net 2))
   (segment (start 132.35 107.95) (end 132.4 108) (width 0.25) (layer F.Cu) (net 2))
@@
   (segment (start 126.16 110.49) (end 125.64 110.49) (width 0.25) (layer F.Cu) (net 6) (status 30))
   (segment (start 136.47 100.33) (end 136.32 100.33) (width 0.25) (layer F.Cu) (net 6) (status 30))
-  (segment (start 136.47 102.58) (end 136.47 100.33) (width 0.25) (layer F.Cu) (net 6) (status 20))
-  (segment (start 132.35 106.7) (end 136.47 102.58) (width 0.25) (layer F.Cu) (net 6))
-  (segment (start 120.6 106.7) (end 132.35 106.7) (width 0.25) (layer F.Cu) (net 6))
-  (segment (start 120.52001 106.77999) (end 120.6 106.7) (width 0.25) (layer F.Cu) (net 6))
-  (segment (start 120.52001 112.22001) (end 120.52001 106.77999) (width 0.25) (layer F.Cu) (net 6))
+  (segment (start 136.47 102.58) (end 136.47 102.58) (width 0.25) (layer F.Cu) (net 6) (status 20))
   (segment (start 124.565 110.49) (end 123.75 111.305) (width 0.25) (layer F.Cu) (net 6))
   (segment (start 125.64 110.49) (end 124.565 110.49) (width 0.25) (layer F.Cu) (net 6) (status 10))
-  (segment (start 123.75 111.305) (end 123.75 112.65) (width 0.25) (layer F.Cu) (net 6))
-  (segment (start 123.75 112.65) (end 123.25 113.15) (width 0.25) (layer F.Cu) (net 6))
-  (segment (start 123.25 113.15) (end 121.45 113.15) (width 0.25) (layer F.Cu) (net 6))
-  (segment (start 121.45 113.15) (end 120.52001 112.22001) (width 0.25) (layer F.Cu) (net 6))
+  (segment (start 136.47 102.58) (end 136.47 100.33) (width 0.25) (layer F.Cu) (net 6) (status 20))
+  (via (at 136.47 102.58) (size 0.8) (drill 0.4) (layers F.Cu B.Cu) (net 6))
+  (segment (start 123.75 111.305) (end 123.75 111.305) (width 0.25) (layer F.Cu) (net 6))
+  (via (at 123.75 111.305) (size 0.8) (drill 0.4) (layers F.Cu B.Cu) (net 6))
+  (segment (start 132.475 102.58) (end 136.47 102.58) (width 0.25) (layer B.Cu) (net 6))
+  (segment (start 123.75 111.305) (end 132.475 102.58) (width 0.25) (layer B.Cu) (net 6))
   (segment (start 135.993763 116.556237) (end 136.55 116) (width 0.25) (layer F.Cu) (net 7))
   (segment (start 135.52499 117.02501) (end 135.993763 116.556237) (width 0.25) (layer F.Cu) (net 7))
@@
   (segment (start 123.8975 117.7) (end 121.92 115.7225) (width 0.25) (layer F.Cu) (net 7))
   (segment (start 126.9575 117.7) (end 123.8975 117.7) (width 0.25) (layer F.Cu) (net 7))
+  (via (at 133.45 114.35) (size 0.8) (drill 0.4) (layers F.Cu B.Cu) (net 8))
+  (via (at 133.4 109.7) (size 0.8) (drill 0.4) (layers F.Cu B.Cu) (net 8))
   (segment (start 134.068763 108.506237) (end 134.625 107.95) (width 0.25) (layer F.Cu) (net 8))
   (segment (start 133.849999 108.725001) (end 134.068763 108.506237) (width 0.25) (layer F.Cu) (net 8))
