File: HABIV/old_board_submodules/stm_power_sd/STM32.kicad_pcb (KiCad board)
At the start: 4 copper layers, 56 parts, among them J1 Conn_ARM_JTAG_SWD_20, J10 Conn_01x02_Male, J12 Conn_01x03_Male, J13 Conn_01x04_Male, J14 Conn_01x05_Male, J15 Conn_01x08_Male, J2 Micro_SD_Card_Det, J3 Conn_01x16_Male, J4 Conn_01x16_Male, J5 Conn_01x16_Male, J6 Conn_01x02_Male, J7 Conn_01x02_Male, J8 Conn_01x02_Male, J9 Conn_01x11_Male, SW1 SW_DPST_x2, U1 STM32F401RET6, U2 TPS564208, U3 TPS564208, Y1 32.768MHz

Commit message: finish submodules and combine
Parts:
- removed 0k1: R1, Resistors_SMD:R_0603_HandSoldering
- removed 0k2: R2, Resistors_SMD:R_0603_HandSoldering
- removed C1: 4.3pF, Capacitors_SMD:C_0603_HandSoldering
- removed C18, C21: 47uF, Capacitors_SMD:C_0603_HandSoldering
- removed C19: 10uF, Capacitors_SMD:C_0603_HandSoldering
- removed C20: 100nF, Capacitors_SMD:C_0603_HandSoldering
- removed D4, D5: LED, LEDs:LED_0603_HandSoldering
- removed J10, J8: Conn_01x02_Male, Pin_Headers:Pin_Header_Straight_1x02_Pitch2.54mm
- removed J12: Conn_01x03_Male, Pin_Headers:Pin_Header_Straight_1x03_Pitch2.54mm
- removed J13: Conn_01x04_Male, Pin_Headers:Pin_Header_Straight_1x04_Pitch2.54mm
- removed J14: Conn_01x05_Male, Pin_Headers:Pin_Header_Straight_1x05_Pitch2.54mm
- removed J15: Conn_01x08_Male, Pin_Headers:Pin_Header_Straight_1x08_Pitch2.54mm
- removed J3: Conn_01x16_Male, Pin_Headers:Pin_Header_Straight_1x16_Pitch2.54mm
- added 10k4: R8, Resistor_SMD:R_0805_2012Metric, F.Cu at (132.3, 84.7)
- added C13: 100nF, Capacitor_SMD:C_0805_2012Metric, F.Cu at (48.8, 104.3)
- added C14: 100nF, Capacitor_SMD:C_0805_2012Metric, F.Cu at (92.9, 84.3)
- added C3: 4.3pF, Capacitor_SMD:C_0805_2012Metric, F.Cu at (134.6, 99.4)
- added C8: 10uF, Capacitor_SMD:C_0805_2012Metric, F.Cu at (57.7, 100.5)
- added C9: 10uF, Capacitor_SMD:C_0805_2012Metric, F.Cu at (84.5, 88.2)
- added D2: LED, LED_SMD:LED_0805_2012Metric, F.Cu at (48.5, 92.2)
- added D3: LED, LED_SMD:LED_0805_2012Metric, F.Cu at (93.2, 96.4)
- added R100: 0k1, Resistor_SMD:R_0805_2012Metric, F.Cu at (138.5, 94.6)
- added R101: 0k2, Resistor_SMD:R_0805_2012Metric, F.Cu at (138.5, 96.1)
- added R13: 0, Resistor_SMD:R_0805_2012Metric, F.Cu at (190.1, 68.8)
- added R14: 0, Resistor_SMD:R_0805_2012Metric, F.Cu at (190.1, 71.2)
- added R15: 0, Resistor_SMD:R_0805_2012Metric, F.Cu at (190.1, 75.8)
- added R18: 0, Resistor_SMD:R_0805_2012Metric, F.Cu at (125.1, 107.5)
- added R38: 33.2k, Resistor_SMD:R_0805_2012Metric, F.Cu at (48.5, 96.3)
- added R39: 10k, Resistor_SMD:R_0805_2012Metric, F.Cu at (47.4, 99.4)
- added R4: 0, Resistor_SMD:R_0805_2012Metric, F.Cu at (190.1, 78.1)
- added R40: 56.2k, Resistor_SMD:R_0805_2012Metric, F.Cu at (93.2, 92.4)
- added R41: 10k, Resistor_SMD:R_0805_2012Metric, F.Cu at (94.2, 89.3)
- added R42: 4.7k, Resistor_SMD:R_0805_2012Metric, F.Cu at (47.4, 89.4)
- added R43: 4.7k, Resistor_SMD:R_0805_2012Metric, F.Cu at (94.3, 99.4)
- 100nF1, 100nF2, 100nF3, 100nF4, 100nF5, 10nF1, 1uF1, 1uF2, 1uF3, 1uF4, 1uF5, 4.7uF1, C2: footprint Capacitors_SMD:C_0603_HandSoldering -> Capacitor_SMD:C_0805_2012Metric
- 10k1: value R6 -> R5; footprint Resistors_SMD:R_0603_HandSoldering -> Resistor_SMD:R_0805_2012Metric
- 10k2: value R7 -> R6; footprint Resistors_SMD:R_0603_HandSoldering -> Resistor_SMD:R_0805_2012Metric
- 10k3: value R8 -> R7; footprint Resistors_SMD:R_0603_HandSoldering -> Resistor_SMD:R_0805_2012Metric
- 22uH1: footprint Inductors_SMD:L_0603_HandSoldering -> Inductor_SMD:L_0805_2012Metric
- C16: value 10uF -> 47uF; footprint Capacitors_SMD:C_0603_HandSoldering -> Capacitor_SMD:C_0805_2012Metric
- C17: value 100nF -> 47uF; footprint Capacitors_SMD:C_0603_HandSoldering -> Capacitor_SMD:C_0805_2012Metric
- J1: value Conn_ARM_JTAG_SWD_20 -> Micro_SD_Card_Det; footprint Pin_Headers:Pin_Header_Straight_2x10_Pitch2.54mm -> Connector_Card:microSD_HC_Hirose_DM3BT-DSF-PEJS
- J2: value Micro_SD_Card_Det -> Conn_ARM_JTAG_SWD_20; footprint Connectors_Card:Hirose_DM3BT-DSF-PEJS -> Connector_PinHeader_2.54mm:PinHeader_2x10_P2.54mm_Vertical
- J4: footprint Pin_Headers:Pin_Header_Straight_1x16_Pitch2.54mm -> Connector_PinHeader_2.54mm:PinHeader_1x16_P2.54mm_Vertical
- J5: value Conn_01x16_Male -> Conn_01x02_Male; footprint Pin_Headers:Pin_Header_Straight_1x16_Pitch2.54mm -> Connector_PinHeader_2.54mm:PinHeader_1x02_P2.54mm_Vertical
- J6, J7: value Conn_01x02_Male -> Conn_01x16_Male; footprint Pin_Headers:Pin_Header_Straight_1x02_Pitch2.54mm -> Connector_PinHeader_2.54mm:PinHeader_1x16_P2.54mm_Vertical
- J9: value Conn_01x11_Male -> Conn_01x02_Male; footprint Pin_Headers:Pin_Header_Straight_1x11_Pitch2.54mm -> Connector_PinHeader_2.54mm:PinHeader_1x02_P2.54mm_Vertical
- R10, R9: value 4.7k -> 56k; footprint Resistors_SMD:R_0603_HandSoldering -> Resistor_SMD:R_0805_2012Metric
- R5, R7: value 10k -> 56k; footprint Resistors_SMD:R_0603_HandSoldering -> Resistor_SMD:R_0805_2012Metric
- R6: value 33.2k -> 56k; footprint Resistors_SMD:R_0603_HandSoldering -> Resistor_SMD:R_0805_2012Metric
- R8: value 56.2k -> 0; footprint Resistors_SMD:R_0603_HandSoldering -> Resistor_SMD:R_0805_2012Metric
- SW1: footprint Buttons_Switches_SMD:SW_SPST_B3U-1000P -> Button_Switch_SMD:SW_SPST_B3U-1000P
- Y1: footprint Crystals:Crystal_SMD_0603-4pin_6.0x3.5mm_HandSoldering -> Crystal:Crystal_SMD_0603-4Pin_6.0x3.5mm_HandSoldering
- moved C16 152.5 mm to (58.6, 116.6), turned to 90 degrees
- moved L3 152.3 mm to (51.4, 109.9)
- moved L4 152.3 mm to (90.2, 78.7)
- moved U5 152.3 mm to (89.7, 88.2)
- moved U4 152.3 mm to (51.8, 100.5)
- moved C17 121.1 mm to (83.9, 71.9), turned to 270 degrees
- moved J7 101.8 mm to (128.3, 117.6), turned to 90 degrees
- moved J1 96.8 mm to (210.9, 74.8), turned to 90 degrees
- moved J6 66.9 mm to (166.6, 72.4), turned to 270 degrees
- moved R9 58.6 mm to (197.8, 65.2)
- moved R8 57.9 mm to (190.1, 73.5), turned to 180 degrees
- moved R7 52.0 mm to (195.6, 77.4), turned to 270 degrees
- moved J2 42.6 mm to (119.8, 107.5), turned to 180 degrees
- moved J4 42.1 mm to (172.6, 114.1), turned to 180 degrees
- moved R6 29.4 mm to (202.2, 65.2), turned to 0 degrees
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- renumbered L2 to L3, L3 to L4, U2 to U4, U3 to U5
Connections:
- 10k1 pad 1: GND -> Net-(10k1-Pad1)
- 10k1 pad 2: Net-(10k1-Pad2) -> GND
- 10k4 pad 1: Net-(10k4-Pad1) -> (no net)
- C16 pad 1: Net-(C16-Pad1) -> +3V3
- C16 pad 2: Net-(C16-Pad2) -> GND
- C17 pad 1: Net-(C17-Pad1) -> +5V
- C17 pad 2: Net-(C17-Pad2) -> GND
- C2 pad 1: Net-(0k2-Pad2) -> Net-(C2-Pad1)
- J1 pad 1: +3V3 -> Net-(J1-Pad1)
- J1 pad 10: GND -> (no net)
- J1 pad 11: Net-(10k1-Pad2) -> GND
- J1 pad 2: +3V3 -> Net-(J1-Pad2)
- J1 pad 3: PB4 -> Net-(J1-Pad3)
- J1 pad 4: GND -> Net-(J1-Pad4)
- J1 pad 5: PA15 -> Net-(J1-Pad5)
- J1 pad 7: PA13 -> Net-(J1-Pad7)
- J1 pad 8: GND -> Net-(J1-Pad8)
- J1 pad 9: PA14 -> (no net)
- J2 pad 10: Net-(J2-Pad10) -> GND
- J2 pad 11: Net-(J2-Pad11) -> Net-(10k2-Pad2)
- J2 pad 2: Net-(J2-Pad2) -> Net-(J2-Pad1)
- J2 pad 3: Net-(J2-Pad3) -> PB4
- J2 pad 4: Net-(J2-Pad4) -> GND
- J2 pad 5: Net-(J2-Pad5) -> PA15
- J2 pad 6: Net-(J2-Pad6) -> GND
- J2 pad 7: Net-(J2-Pad7) -> PA13
- J2 pad 8: Net-(J2-Pad8) -> GND
- J2 pad 9: Net-(J2-Pad9) -> PA14
- J4 pad 1: PB0 -> PA0
- J4 pad 10: PB9 -> PA9
- J4 pad 11: PB10 -> PA10
- J4 pad 12: PB11 -> PA11
- J4 pad 13: PB12 -> PA12
- J4 pad 14: PB13 -> PA13
- J4 pad 15: PB14 -> PA14
- J4 pad 16: PB15 -> PA15
- J4 pad 2: PB1 -> PA1
- J4 pad 3: PB2 -> PA2
- J4 pad 4: PB3 -> PA3
- J4 pad 5: PB4 -> PA4
- J4 pad 6: PB5 -> PA5
- J4 pad 7: PB6 -> PA6
- J4 pad 8: PB7 -> PA7
- J4 pad 9: PB8 -> PA8
- J5 pad 1: PC0 -> GND
- J5 pad 2: PC1 -> +3V3
- J6 pad 1: GND -> PB0
- J6 pad 2: +3V3 -> PB1
- J7 pad 1: Net-(C16-Pad1) -> PC0
- J7 pad 2: Net-(C16-Pad2) -> PC1
- J9 pad 1: Net-(J2-Pad1) -> Net-(C8-Pad1)
- J9 pad 2: Net-(J2-Pad2) -> GND
- L3 pad 1: Net-(C18-Pad1) -> +3V3
- L3 pad 2: Net-(C17-Pad1) -> Net-(C13-Pad1)
- L4 pad 1: Net-(C21-Pad1) -> +5V
- R10 pad 1: Net-(C16-Pad2) -> Net-(J1-Pad4)
- R10 pad 2: Net-(D5-Pad1) -> Net-(J1-Pad8)
- R5 pad 1: Net-(C16-Pad2) -> Net-(J1-Pad4)
- R5 pad 2: Net-(R5-Pad2) -> Net-(J1-Pad1)
- R6 pad 1: Net-(R5-Pad2) -> Net-(J1-Pad4)
- R6 pad 2: Net-(C18-Pad1) -> Net-(J1-Pad2)
- R7 pad 1: Net-(C16-Pad2) -> Net-(J1-Pad3)
- R7 pad 2: Net-(R7-Pad2) -> Net-(J1-Pad4)
- R8 pad 1: Net-(R7-Pad2) -> Net-(J1-Pad5)
- R8 pad 2: Net-(C21-Pad1) -> PA5
- R9 pad 1: Net-(C16-Pad2) -> Net-(J1-Pad4)
- R9 pad 2: Net-(D4-Pad1) -> Net-(J1-Pad7)
- U1 pad 5: Net-(U1-Pad5) -> (no net)
- U1 pad 6: Net-(U1-Pad6) -> (no net)
- U1 pad 60: Net-(10k4-Pad1) -> Net-(10k1-Pad1)
- U4 pad 1: Net-(C16-Pad2) -> GND
- U4 pad 2: Net-(C17-Pad1) -> Net-(C13-Pad1)
- U4 pad 3: Net-(C16-Pad1) -> Net-(C8-Pad1)
- U4 pad 4: Net-(R5-Pad2) -> Net-(R38-Pad1)
- U4 pad 5: Net-(C16-Pad1) -> Net-(C8-Pad1)
- U4 pad 6: Net-(C17-Pad2) -> Net-(C13-Pad2)
- U5 pad 1: Net-(C16-Pad2) -> GND
- U5 pad 3: Net-(C16-Pad1) -> Net-(C8-Pad1)
- U5 pad 4: Net-(R7-Pad2) -> Net-(R40-Pad1)
- U5 pad 5: Net-(C16-Pad1) -> Net-(C8-Pad1)
- Y1 pad 1: Net-(0k1-Pad2) -> Net-(C2-Pad1)
- Y1 pad 4: Net-(0k2-Pad2) -> Net-(C3-Pad1)
Routing:
- net GND: track 103.5 -> 360.1 mm, vias 18 -> 105
- net Net-(C16-Pad2): track 206.2 -> 0.00 mm, vias 87 -> 0
- net Net-(J2-Pad11): track 54.3 -> 0.00 mm
- net +3V3: track 93.9 -> 135.8 mm, vias 10 -> 12
- net Net-(C18-Pad1): track 35.8 -> 0.00 mm, vias 1 -> 0
- net Net-(C8-Pad1): track 0.00 -> 33.3 mm, vias 0 -> 4
- net Net-(C16-Pad1): track 33.3 -> 0.00 mm, vias 4 -> 0
- net Net-(J2-Pad10): track 32.7 -> 0.00 mm
- net Net-(J1-Pad2): track 0.00 -> 31.4 mm, vias 0 -> 4
- net Net-(J1-Pad4): track 0.00 -> 30.4 mm, vias 0 -> 2
- net Net-(J1-Pad7): track 0.00 -> 18.9 mm, vias 0 -> 2
- net Net-(10k1-Pad2): track 16.2 -> 0.00 mm
- net Net-(J2-Pad2): track 13.1 -> 0.00 mm
- net Net-(J1-Pad3): track 0.00 -> 12.9 mm
- net Net-(J2-Pad3): track 12.5 -> 0.00 mm
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- added copper zone on B.Cu, net Net-(C20-Pad1)
- added copper zone on F.Cu, net Net-(C20-Pad1)
- removed copper zone on B.Cu, net Net-(C14-Pad1)
- removed copper zone on F.Cu, net Net-(C14-Pad1)
Other:
- board text removed: "CLK"
- board text removed: "CMD"
- board text removed: "DAT0"
- board text removed: "DAT1"
- board text removed: "DAT2"
- board text removed: "DAT3"
- board text removed: "DETA"
- board text removed: "DETB"
- board text removed: "SHLD"
- board text removed: "VDD"
- board text removed: "VSS"
