File: HABIV/old_board_submodules/stm_power_sd/STM32.sch (KiCad schematic (older format))
At the start: 56 parts, among them J1 Conn_ARM_JTAG_SWD_20, J10 Conn_01x02_Male, J12 Conn_01x03_Male, J13 Conn_01x04_Male, J14 Conn_01x05_Male, J15 Conn_01x08_Male, J2 Micro_SD_Card_Det, J3 Conn_01x16_Male, J4 Conn_01x16_Male, J5 Conn_01x16_Male, J6 Conn_01x02_Male, J7 Conn_01x02_Male, J8 Conn_01x02_Male, J9 Conn_01x11_Male, SW1 SW_DPST_x2, U1 STM32F401RET6, U2 TPS564208, U3 TPS564208, Y1 32.768MHz

Commit message: finish submodules and combine
Parts:
- removed 0k1: R1, Resistors_SMD:R_0603_HandSoldering, symbol STM32-rescue:R
- removed 0k2: R2, Resistors_SMD:R_0603_HandSoldering, symbol STM32-rescue:R
- removed J10, J8: Conn_01x02_Male, Pin_Headers:Pin_Header_Straight_1x02_Pitch2.54mm, symbol STM32-rescue:Conn_01x02_Male
- removed J12: Conn_01x03_Male, Pin_Headers:Pin_Header_Straight_1x03_Pitch2.54mm, symbol STM32-rescue:Conn_01x03_Male
- removed J13: Conn_01x04_Male, Pin_Headers:Pin_Header_Straight_1x04_Pitch2.54mm, symbol STM32-rescue:Conn_01x04_Male
- removed J14: Conn_01x05_Male, Pin_Headers:Pin_Header_Straight_1x05_Pitch2.54mm, symbol STM32-rescue:Conn_01x05_Male
- removed J15: Conn_01x08_Male, Pin_Headers:Pin_Header_Straight_1x08_Pitch2.54mm, symbol STM32-rescue:Conn_01x08_Male
- removed J9: Conn_01x11_Male, Pin_Headers:Pin_Header_Straight_1x11_Pitch2.54mm, symbol STM32-rescue:Conn_01x11_Male
- added R10, R5, R6, R7, R9: 56k, Resistor_SMD:R_0805_2012Metric, symbol Device:R_Small
- added R100: 0k1, Resistor_SMD:R_0805_2012Metric, symbol Device:R_Small
- added R101: 0k2, Resistor_SMD:R_0805_2012Metric, symbol Device:R_Small
- added R13, R14, R15, R18, R4, R8: 0, Resistor_SMD:R_0805_2012Metric, symbol Device:R
- 100nF1, 100nF2, 100nF3, 100nF4, 100nF5, 10nF1, 1uF1, 1uF2, 1uF3, 1uF4, 1uF5, 4.7uF1: footprint Capacitors_SMD:C_0603_HandSoldering -> Capacitor_SMD:C_0805_2012Metric; symbol STM32-rescue:C -> STM32-rescue:C-STM32-rescue-habiv-board-rescue
- 10k1: renamed from 10k4; footprint Resistors_SMD:R_0603_HandSoldering -> Resistor_SMD:R_0805_2012Metric; symbol STM32-rescue:R -> STM32-rescue:R-STM32-rescue-habiv-board-rescue
- 10k2: renamed from 10k1; footprint Resistors_SMD:R_0603_HandSoldering -> Resistor_SMD:R_0805_2012Metric; symbol STM32-rescue:R -> STM32-rescue:R-STM32-rescue-habiv-board-rescue
- 10k3: renamed from 10k2; footprint Resistors_SMD:R_0603_HandSoldering -> Resistor_SMD:R_0805_2012Metric; symbol STM32-rescue:R -> STM32-rescue:R-STM32-rescue-habiv-board-rescue
- 10k4: renamed from 10k3; footprint Resistors_SMD:R_0603_HandSoldering -> Resistor_SMD:R_0805_2012Metric; symbol STM32-rescue:R -> STM32-rescue:R-STM32-rescue-habiv-board-rescue
- 22uH1: footprint Inductors_SMD:L_0603_HandSoldering -> Inductor_SMD:L_0805_2012Metric; symbol STM32-rescue:L -> STM32-rescue:L-STM32-rescue-habiv-board-rescue
- C13: renamed from C17; footprint Capacitors_SMD:C_0603_HandSoldering -> Capacitor_SMD:C_0805_2012Metric; symbol STM32-rescue:C -> STM32-rescue:C-STM32-rescue-habiv-board-rescue
- C14: renamed from C20; footprint Capacitors_SMD:C_0603_HandSoldering -> Capacitor_SMD:C_0805_2012Metric; symbol STM32-rescue:C -> STM32-rescue:C-STM32-rescue-habiv-board-rescue
- C16: renamed from C18; footprint Capacitors_SMD:C_0603_HandSoldering -> Capacitor_SMD:C_0805_2012Metric; symbol STM32-rescue:C -> STM32-rescue:C-STM32-rescue-habiv-board-rescue
- C17: renamed from C21; footprint Capacitors_SMD:C_0603_HandSoldering -> Capacitor_SMD:C_0805_2012Metric; symbol STM32-rescue:C -> STM32-rescue:C-STM32-rescue-habiv-board-rescue
- C2: renamed from C1; footprint Capacitors_SMD:C_0603_HandSoldering -> Capacitor_SMD:C_0805_2012Metric; symbol STM32-rescue:C -> STM32-rescue:C-STM32-rescue-habiv-board-rescue
- C3: renamed from C2; footprint Capacitors_SMD:C_0603_HandSoldering -> Capacitor_SMD:C_0805_2012Metric; symbol STM32-rescue:C -> STM32-rescue:C-STM32-rescue-habiv-board-rescue
- C8: renamed from C16; footprint Capacitors_SMD:C_0603_HandSoldering -> Capacitor_SMD:C_0805_2012Metric; symbol STM32-rescue:C -> STM32-rescue:C-STM32-rescue-habiv-board-rescue
- C9: renamed from C19; footprint Capacitors_SMD:C_0603_HandSoldering -> Capacitor_SMD:C_0805_2012Metric; symbol STM32-rescue:C -> STM32-rescue:C-STM32-rescue-habiv-board-rescue
- D2: renamed from D5; footprint LEDs:LED_0603_HandSoldering -> LED_SMD:LED_0805_2012Metric; symbol STM32-rescue:LED -> STM32-rescue:LED-STM32-rescue-habiv-board-rescue
- D3: renamed from D4; footprint LEDs:LED_0603_HandSoldering -> LED_SMD:LED_0805_2012Metric; symbol STM32-rescue:LED -> STM32-rescue:LED-STM32-rescue-habiv-board-rescue
- J1: renamed from J2; footprint Connectors_Card:Hirose_DM3BT-DSF-PEJS -> Connector_Card:microSD_HC_Hirose_DM3BT-DSF-PEJS; symbol STM32-rescue:Micro_SD_Card_Det -> STM32-rescue:Micro_SD_Card_Det-STM32-rescue-habiv-board-rescue
- J2: renamed from J1; footprint Pin_Headers:Pin_Header_Straight_2x10_Pitch2.54mm -> Connector_PinHeader_2.54mm:PinHeader_2x10_P2.54mm_Vertical; symbol STM32-rescue:Conn_ARM_JTAG_SWD_20 -> STM32-rescue:Conn_ARM_JTAG_SWD_20-STM32-rescue-habiv-board-rescue
- J4: renamed from J3; footprint Pin_Headers:Pin_Header_Straight_1x16_Pitch2.54mm -> Connector_PinHeader_2.54mm:PinHeader_1x16_P2.54mm_Vertical; symbol STM32-rescue:Conn_01x16_Male -> STM32-rescue:Conn_01x16_Male-STM32-rescue-habiv-board-rescue
- J5: renamed from J6; footprint Pin_Headers:Pin_Header_Straight_1x02_Pitch2.54mm -> Connector_PinHeader_2.54mm:PinHeader_1x02_P2.54mm_Vertical; symbol STM32-rescue:Conn_01x02_Male -> STM32-rescue:Conn_01x02_Male-STM32-rescue-habiv-board-rescue
- J6: renamed from J4; footprint Pin_Headers:Pin_Header_Straight_1x16_Pitch2.54mm -> Connector_PinHeader_2.54mm:PinHeader_1x16_P2.54mm_Vertical; symbol STM32-rescue:Conn_01x16_Male -> STM32-rescue:Conn_01x16_Male-STM32-rescue-habiv-board-rescue
- J7: renamed from J5; footprint Pin_Headers:Pin_Header_Straight_1x16_Pitch2.54mm -> Connector_PinHeader_2.54mm:PinHeader_1x16_P2.54mm_Vertical; symbol STM32-rescue:Conn_01x16_Male -> STM32-rescue:Conn_01x16_Male-STM32-rescue-habiv-board-rescue
- J9: renamed from J7; footprint Pin_Headers:Pin_Header_Straight_1x02_Pitch2.54mm -> Connector_PinHeader_2.54mm:PinHeader_1x02_P2.54mm_Vertical; symbol STM32-rescue:Conn_01x02_Male -> STM32-rescue:Conn_01x02_Male-STM32-rescue-habiv-board-rescue
- L3: renamed from L2; symbol STM32-rescue:L -> STM32-rescue:L-STM32-rescue-habiv-board-rescue
- L4: renamed from L3; symbol STM32-rescue:L -> STM32-rescue:L-STM32-rescue-habiv-board-rescue
- R38: renamed from R6; footprint Resistors_SMD:R_0603_HandSoldering -> Resistor_SMD:R_0805_2012Metric; symbol STM32-rescue:R -> STM32-rescue:R-STM32-rescue-habiv-board-rescue
- R39: renamed from R5; footprint Resistors_SMD:R_0603_HandSoldering -> Resistor_SMD:R_0805_2012Metric; symbol STM32-rescue:R -> STM32-rescue:R-STM32-rescue-habiv-board-rescue
- R40: renamed from R8; footprint Resistors_SMD:R_0603_HandSoldering -> Resistor_SMD:R_0805_2012Metric; symbol STM32-rescue:R -> STM32-rescue:R-STM32-rescue-habiv-board-rescue
- R41: renamed from R7; footprint Resistors_SMD:R_0603_HandSoldering -> Resistor_SMD:R_0805_2012Metric; symbol STM32-rescue:R -> STM32-rescue:R-STM32-rescue-habiv-board-rescue
- R42: renamed from R10; footprint Resistors_SMD:R_0603_HandSoldering -> Resistor_SMD:R_0805_2012Metric; symbol STM32-rescue:R -> STM32-rescue:R-STM32-rescue-habiv-board-rescue
- R43: renamed from R9; footprint Resistors_SMD:R_0603_HandSoldering -> Resistor_SMD:R_0805_2012Metric; symbol STM32-rescue:R -> STM32-rescue:R-STM32-rescue-habiv-board-rescue
- SW1: footprint Buttons_Switches_SMD:SW_SPST_B3U-1000P -> Button_Switch_SMD:SW_SPST_B3U-1000P; symbol STM32-rescue:SW_DPST_x2 -> STM32-rescue:SW_DPST_x2-STM32-rescue-habiv-board-rescue
- U1: symbol STM32-rescue:STM32F401RET6 -> STM32-rescue:STM32F401RET6-STM32-rescue-habiv-board-rescue
- U4: renamed from U2; symbol STM32-rescue:TPS564208 -> STM32-rescue:TPS564208-STM32-rescue-habiv-board-rescue
- U5: renamed from U3; symbol STM32-rescue:TPS564208 -> STM32-rescue:TPS564208-STM32-rescue-habiv-board-rescue
- Y1: footprint Crystals:Crystal_SMD_0603-4pin_6.0x3.5mm_HandSoldering -> Crystal:Crystal_SMD_0603-4Pin_6.0x3.5mm_HandSoldering; symbol STM32-rescue:Crystal_GND23 -> STM32-rescue:Crystal_GND23-STM32-rescue-habiv-board-rescue
Connections:
- net +3V3: now also C16.1, D2.2 (A), L3.1, R38.2, R18.1, R4.1; no longer J2.1 (VTREF), J2.2 (VCC/NC)
- net GND: now also C16.2, C17.2, C8.2, C9.2, J1.11 (SHIELD), J1.6 (VSS), J9.2 (Pin_2), R39.1, R41.1, R42.1, R43.1, U4.1 (GND), U5.1 (GND)
- net PA5: now also R8.2
- net PA6: now also R14.2
- net PA7: now also R15.1
- net PA9: now also R13.1
- net at U1.3 (PC14): now also R100.1
- net at U1.4 (PC15): now also R101.1
- net at C2.1, Y1.1: now also R100.2
- net at C3.1, Y1.4: now also R101.2
- net at J1.1 (DAT2): now also R5.2
- net at J1.2 (DAT3/CD): now also R13.2, R6.2
- net at J1.3 (CMD): now also R15.2, R7.1
- net at J1.4 (VDD): now also R10.1, R4.2, R5.1, R6.1, R7.2, R9.1
- net at J1.5 (CLK): now also R8.1
- net at J1.7 (DAT0): now also R14.1, R9.2
- net at J1.8 (DAT1): now also R10.2
- net +5V: now reaches C17.1, D3.2 (A), L4.1, R40.2
- new net: J2.1 (VTREF), J2.2 (VCC/NC), R18.2
- no-connect marks 0 -> 2
Other:
- moved on the sheet: 100nF1, 100nF2, 100nF3, 100nF4, 100nF5, 10k1, 10k2, 10k3, 10k4, 10nF1, 1uF1, 1uF2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
