File: HABIV/habiv-board/_autosave-habiv-board.kicad_pcb (KiCad board)
At the start: 4 copper layers, 100.3 x 120.9 mm, 126 parts, among them IC1 RTC_PCF8523T, J1 Micro_SD_Card_Det, J10 Conn_01x02_Female, J11 Conn_01x02_Female, J12 Conn_01x02_Female, J13 Conn_01x02_Female, J14 Conn_01x02_Female, J15 Conn_01x02_Female, J16 Conn_01x02_Female, J18 Conn_01x03_Male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

Commit message: Updates for rn
Parts:
- removed JP7: Jumper, Connector_PinHeader_2.54mm:PinHeader_1x02_P2.54mm_Vertical
- removed R16: 1K, Resistor_SMD:R_0805_2012Metric
- C4: value 10u -> 3.3uF
- moved JP6 130.6 mm to (176.7, 36.7)
- moved C1 2.29 mm to (173.5, 38.0)
- moved C4 2.29 mm to (171.2, 38.0)
Connections:
- B2 pad 1: Net-(B2-Pad1) -> GND
- IC1 pad 4: Net-(B2-Pad1) -> GND
- IC1 pad 8: Net-(IC1-Pad8) -> Net-(C4-Pad1)
- JP6 pad 1: Net-(B2-Pad1) -> Net-(JP6-Pad1)
- JP6 pad 2: GND -> +3V3
- R2 pad 1: Net-(IC1-Pad8) -> +3V3
- R3 pad 1: Net-(IC1-Pad8) -> +3V3
- U3 pad P$13: (no net) -> Net-(U3-PadP$13)
- U3 pad P$14: (no net) -> Net-(U3-PadP$14)
- U3 pad P$15: (no net) -> Net-(U3-PadP$15)
- U3 pad P$16: (no net) -> Net-(U3-PadP$16)
- U3 pad P$17: (no net) -> Net-(U3-PadP$17)
- U3 pad P$18: (no net) -> Net-(U3-PadP$18)
- U3 pad P$2: (no net) -> Net-(U3-PadP$2)
- U3 pad P$20: (no net) -> Net-(U3-PadP$20)
- U3 pad P$4: (no net) -> Net-(U3-PadP$4)
- U3 pad P$6: (no net) -> Net-(U3-PadP$6)
- U3 pad P$7: (no net) -> Net-(U3-PadP$7)
Routing:
- net Net-(C4-Pad1): track 23.3 -> 10.3 mm, vias 2 -> 1
- net Net-(C1-Pad1): track 6.49 -> 0.00 mm, vias 2 -> 0
- net +3V3: track 71.8 -> 65.6 mm
- net Net-(IC1-Pad8): track 13.5 -> 8.16 mm
- net Net-(B2-Pad1): track 3.41 -> 0.00 mm, vias 1 -> 0
- net GND: track 326.7 -> 330.1 mm, vias 138 -> 139
