File: HABIV/habiv-board/_autosave-habiv-board.sch (KiCad schematic (older format))
At the start: 123 parts, among them IC1 RTC_PCF8523T, J1 Micro_SD_Card_Det, J10 Conn_01x02_Female, J11 Conn_01x02_Female, J12 Conn_01x02_Female, J13 Conn_01x02_Female, J14 Conn_01x02_Female, J15 Conn_01x02_Female, J16 Conn_01x02_Female, J18 Conn_01x03_Male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

Commit message: Updates for rn
Parts:
- C4: value 10u -> 3.3uF
- R16: footprint (none) -> Resistor_SMD:R_0805_2012Metric
Changed lines of the file:
@@
 P 2850 2400
 F 0 "C4" H 2942 2446 50  0000 L CNN
-F 1 "10u" H 2942 2355 50  0000 L CNN
+F 1 "3.3uF" H 2942 2355 50  0000 L CNN
 F 2 "Capacitor_SMD:C_0805_2012Metric" H 2850 2400 50  0001 C CNN
 F 3 "~" H 2850 2400 50  0001 C CNN
@@
 F 0 "R16" H 2920 1946 50  0000 L CNN
 F 1 "1K" H 2920 1855 50  0000 L CNN
-F 2 "" V 2780 1900 50  0001 C CNN
+F 2 "Resistor_SMD:R_0805_2012Metric" V 2780 1900 50  0001 C CNN
 F 3 "~" H 2850 1900 50  0001 C CNN
 	1    2850 1900
